File: Hardware/Mainboard/2.0.2/AirMQ - 2.0.2.kicad_sch (KiCad schematic)
At the start: 61 parts, among them J2 I2C, J2 MAIN_PWR, J3 EXT, J4 UART, J5 SEN5x, J6 1Wire/LED, J6 USB_C, SW1 RESET, SW2 BOOT, U1 SCD40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

Commit message: added schematic pdf
Parts:
- C14: value 0.1 uF -> DNP
- D1: footprint Diode_SMD:D_1210_3225Metric -> Diode_SMD:D_SMA
- D3: LCSC (none) -> C2909963
- J5: footprint Connector_JST:JST_GH_BM06B-GHS-TBT_1x06-1MP_P1.25mm_Vertical -> Connector_JST:JST_GH_SM06B-GHS-TB_1x06-1MP_P1.25mm_Horizontal
- R10: value 10k -> 100k
Connections:
- net VCC is gone; now on net +3V3: C1.1, C25.1, C3.1, D1.1 (A1), F2.1, R21.1, U7.5 (VIN)
- net +3V3: now also J2.2 (Pin_2); no longer J2.1 (Pin_1)
- net GND: now also J2.1 (Pin_1); no longer J2.2 (Pin_2)
- net SCL: now also J2.3 (Pin_3); no longer J2.4 (Pin_4)
- net SDA: now also J2.4 (Pin_4); no longer J2.3 (Pin_3)
Other:
- company: (none) -> MQ Labs
- title: (none) -> AirMQ Air Quality sensor
Changed lines of the file:
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@@
 (kicad_sch (version 20230121) (generator eeschema)
   (paper "A4")
+  (title_block
+    (title "AirMQ Air Quality sensor")
+    (company "MQ Labs")
+  )
   (junction (at 90.17 113.665) (diameter 0) (color 0 0 0 0)
   )
@@
   (junction (at 62.865 156.21) (diameter 0) (color 0 0 0 0)
   )
+  (junction (at 212.725 56.515) (diameter 0) (color 0 0 0 0)
+  )
   (junction (at 73.66 42.545) (diameter 0) (color 0 0 0 0)
   )
@@
   (junction (at 163.195 31.75) (diameter 0) (color 0 0 0 0)
   )
-  (junction (at 212.725 56.515) (diameter 0) (color 0 0 0 0)
-  )
   (junction (at 83.82 85.725) (diameter 0) (color 0 0 0 0)
   )
@@
   (junction (at 46.99 85.725) (diameter 0) (color 0 0 0 0)
   )
+  (junction (at 210.185 48.895) (diameter 0) (color 0 0 0 0)
+  )
   (junction (at 83.82 52.705) (diameter 0) (color 0 0 0 0)
   )
@@
   (junction (at 142.875 153.035) (diameter 0) (color 0 0 0 0)
   )
+  (junction (at 210.185 51.435) (diameter 0) (color 0 0 0 0)
+  )
   (junction (at 268.605 42.545) (diameter 0) (color 0 0 0 0)
   )
@@
   (junction (at 221.615 99.06) (diameter 0) (color 0 0 0 0)
   )
-  (junction (at 210.185 48.895) (diameter 0) (color 0 0 0 0)
-  )
   (junction (at 156.845 31.75) (diameter 0) (color 0 0 0 0)
   )
@@
     (stroke (width 0) (type default))
   )
-  (wire (pts (xy 212.725 51.435) (xy 212.725 56.515))
-    (stroke (width 0) (type default))
-  )
   (wire (pts (xy 207.01 56.515) (xy 212.725 56.515))
     (stroke (width 0) (type default))
@@
     (stroke (width 0) (type default))
   )
-  (wire (pts (xy 210.185 48.895) (xy 222.885 48.895))
-    (stroke (width 0) (type default))
-  )
   (wire (pts (xy 194.31 102.235) (xy 187.96 102.235))
     (stroke (width 0) (type default))
@@
     (stroke (width 0) (type default))
   )
+  (wire (pts (xy 210.185 51.435) (xy 210.185 64.77))
+    (stroke (width 0) (type default))
+  )
   (wire (pts (xy 163.83 179.07) (xy 152.4 179.07))
     (stroke (width 0) (type default))
@@
     (stroke (width 0) (type default))
   )
+  (wire (pts (xy 212.725 48.895) (xy 212.725 56.515))
+    (stroke (width 0) (type default))
+  )
   (wire (pts (xy 239.395 156.21) (xy 242.57 156.21))
     (stroke (width 0) (type default))
@@
     (stroke (width 0) (type default))
   )
+  (wire (pts (xy 212.725 48.895) (xy 222.885 48.895))
+    (stroke (width 0) (type default))
+  )
   (wire (pts (xy 80.01 85.725) (xy 83.82 85.725))
     (stroke (width 0) (type default))
@@
     (stroke (width 0) (type default))
   )
-  (wire (pts (xy 215.9 56.515) (xy 222.885 56.515))
+  (wire (pts (xy 216.535 56.515) (xy 222.885 56.515))
     (stroke (width 0) (type default))
   )
@@
     (stroke (width 0) (type default))
   )
-  (wire (pts (xy 212.725 51.435) (xy 222.885 51.435))
-    (stroke (width 0) (type default))
-  )
   (wire (pts (xy 163.195 129.54) (xy 163.195 134.62))
     (stroke (width 0) (type default))
   )
-  (wire (pts (xy 210.185 48.895) (xy 210.185 64.77))
-    (stroke (width 0) (type default))
-  )
   (wire (pts (xy 106.68 160.02) (xy 102.235 160.02))
     (stroke (width 0) (type default))
@@
     (stroke (width 0) (type default))
   )
-  (wire (pts (xy 207.01 48.895) (xy 210.185 48.895))
-    (stroke (width 0) (type default))
-  )
   (wire (pts (xy 246.38 135.89) (xy 245.11 135.89))
     (stroke (width 0) (type default))
@@
     (stroke (width 0) (type default))
   )
+  (wire (pts (xy 210.185 51.435) (xy 222.885 51.435))
+    (stroke (width 0) (type default))
+  )
   (wire (pts (xy 132.08 60.96) (xy 136.525 60.96))
     (stroke (width 0) (type default))
@@
     (stroke (width 0) (type default))
   )
+  (wire (pts (xy 207.01 48.895) (xy 210.185 48.895))
+    (stroke (width 0) (type default))
+  )
   (wire (pts (xy 252.095 52.705) (xy 245.745 52.705))
     (stroke (width 0) (type default))
@@
     (stroke (width 0) (type default))
   )
-  (wire (pts (xy 210.185 41.91) (xy 210.185 48.895))
+  (wire (pts (xy 210.185 48.895) (xy 210.185 51.435))
     (stroke (width 0) (type default))
   )
@@
     (stroke (width 0) (type default))
   )
-  (wire (pts (xy 215.9 53.975) (xy 222.885 53.975))
+  (wire (pts (xy 216.535 53.975) (xy 222.885 53.975))
     (stroke (width 0) (type default))
   )
@@
     (stroke (width 0) (type default))
   )
+  (wire (pts (xy 210.185 41.91) (xy 210.185 48.895))
+    (stroke (width 0) (type default))
+  )
   (wire (pts (xy 133.35 44.45) (xy 133.35 53.34))
     (stroke (width 0) (type default))
@@
     (effects (font (size 1.27 1.27)) (justify right bottom))
   )
-  (label "SCL" (at 215.9 56.515 0) (fields_autoplaced)
+  (label "SDA" (at 216.535 56.515 0) (fields_autoplaced)
     (effects (font (size 1.27 1.27)) (justify left bottom))
   )
-  (label "SDA" (at 215.9 53.975 0) (fields_autoplaced)
+  (label "SCL" (at 216.535 53.975 0) (fields_autoplaced)
     (effects (font (size 1.27 1.27)) (justify left bottom))
   )
@@
     (effects (font (size 1.27 1.27)) (justify right bottom))
   )
+  (label "VCC" (at 216.535 51.435 0) (fields_autoplaced)
+    (effects (font (size 1.27 1.27)) (justify left bottom))
+  )
   (label "IO9" (at 38.1 97.155 0) (fields_autoplaced)
     (effects (font (size 1.27 1.27)) (justify left bottom))
@@
     (effects (font (size 1.27 1.27)) (justify left bottom))
   )
+  (label "GND" (at 216.535 48.895 0) (fields_autoplaced)
+    (effects (font (size 1.27 1.27)) (justify left bottom))
+  )
   (label "SDA" (at 134.62 171.45 0) (fields_autoplaced)
     (effects (font (size 1.27 1.27)) (justify left bottom))
@@
     (effects (font (size 1.27 1.27)) (justify left bottom))
   )
+  (label "VCC" (at 36.195 42.545 0) (fields_autoplaced)
+    (effects (font (size 1.27 1.27)) (justify left bottom))
+  )
   (label "IO4" (at 95.885 177.8 0) (fields_autoplaced)
     (effects (font (size 1.27 1.27)) (justify left bottom))
@@
   (symbol (lib_id "Device:R") (at 133.35 38.735 0) (unit 1)
     (in_bom yes) (on_board yes) (dnp no)
-    (property "Reference" "R4" (at 133.35 34.925 0)
+    (property "Reference" "R4" (at 135.255 36.83 0)
       (effects (font (size 1.27 1.27)) (justify left))
     )
-    (property "Value" "10k" (at 133.35 42.545 0)
+    (property "Value" "10k" (at 135.255 40.005 0)
       (effects (font (size 1.27 1.27)) (justify left))
     )
@@
       (effects (font (size 1.27 1.27)) (justify left))
     )
-    (property "Footprint" "Diode_SMD:D_1210_3225Metric" (at 244.475 93.98 0)
+    (property "Footprint" "Diode_SMD:D_SMA" (at 244.475 93.98 0)
       (effects (font (size 1.27 1.27)) hide)
     )
@@
       (effects (font (size 1.27 1.27)) (justify left))
     )
-    (property "Value" "0.1 uF" (at 197.485 99.695 0)
+    (property "Value" "DNP" (at 194.31 99.06 0)
       (effects (font (size 1.27 1.27)) (justify left))
     )
@@
       (effects (font (size 1.27 1.27)) hide)
     )
+    (property "LCSC" "C2909963" (at 244.475 118.11 90)
+      (effects (font (size 1.27 1.27)) hide)
+    )
     (pin "1")
     (pin "2")
@@
       (effects (font (size 1.27 1.27)) (justify left))
     )
-    (property "Footprint" "Connector_JST:JST_GH_BM06B-GHS-TBT_1x06-1MP_P1.25mm_Vertical" (at 227.965 104.14 0)
+    (property "Footprint" "Connector_JST:JST_GH_SM06B-GHS-TB_1x06-1MP_P1.25mm_Horizontal" (at 227.965 104.14 0)
       (effects (font (size 1.27 1.27)) hide)
     )
@@
       (effects (font (size 1.27 1.27)))
     )
-    (property "Value" "10k" (at 196.85 81.28 0)
+    (property "Value" "100k" (at 198.12 81.915 0)
       (effects (font (size 1.27 1.27)))
     )
